Commit message: Add glim_pcap_rosbag for direct pcap+mcap offline mapping
Lets GLIM consume a Luminar Iris .pcap and an IMU/odom .mcap directly,
avoiding the merge_luminar_pcap.py pre-merge step. The new executable
parses Iris UDP packets in C++ via libpcap, assembles them into the same
PointCloud2 layout the Python merger produced, time-merges with the
mcap reader, and dispatches to the existing GlimROS callbacks.

New:
- glim_ros2/include/glim_ros/iris_pcap_reader.hpp/.cpp - classic-pcap
  reader (rejects pcapng), datalink dispatch (EN10MB/SLL/SLL2/RAW),
  Iris bit-unpack parser, scan assembler with inactivity timeout +
  cross-lidar reorder buffer.
- glim_ros2/include/glim_ros/lidar_concat.hpp - concat helpers extracted
  from glim_rosbag.cpp into a header-only module shared by both
  executables; adds load_aux_sensors_from_config() for the URDF/manual
  transform path.
- glim_ros2/src/glim_pcap_rosbag.cpp - main executable. Time-merged
  dispatch with bag-primary-points guard, additive extension subs,
  /clock publisher (fixes TF_OLD_DATA in viewers via use_sim_time),
  attached spdlog file sink at <dump_path>/run.log.
- glim/config/config_pcap.json + entry in config.json - pcap source
  config (lidar IPs/topics/frames/ports, inactivity_sec, reorder window).

Modified:
- glim_ros2/CMakeLists.txt - libpcap detection + new executable.
- glim_ros2/package.xml - libpcap-dev rosdep.
- glim_ros2/src/glim_rosbag.cpp - refactored to use lidar_concat.hpp;
  behavior unchanged.
- glim_ext/config/config_gnss_global.json - dropped prior_inf_scale
  from 1e4 to 10 (sigma 30cm); soft anchor avoids back-and-forth
  optimization snapping. Switched gnss_topic to /vks/global_odom.
- glim/config/config_ros.json - imu_topic /gps_na/imu, gnss_global
  commented out by default, imu_validator extension added.
- glim/config/config_sensors.json - urdf_imu_frame: novatel_a, manual
  T_lidar_imu fallback; URDF restructure aligned.
- glim/config/config_odometry_gpu.json - commented out hardcoded
  init_T_world_imu / init_v_world_imu (was injecting a 9.5 m/s
  initial velocity at frame 0).
- av24.urdf - sensor frame restructure (gps_antenna_*, novatel_a/b,
  pointonenav, vectornav, imu_top/bottom).

Scripts:
- scripts/plot_imu_dups.py - per-IMU duplicate-stamp diagnostic plot.
- scripts/plot_imu_window.py - zoomed recv/header.stamp window plot.
- scripts/extract_init_velocity.py - pull initial v_world_imu prior
  from a rosbag for the URDF init path.
- merge_luminar_pcap.py - the original Python reference merger,
  tracked for historical reference.

Run:
  ROS_DOMAIN_ID=99 ros2 run glim_ros glim_pcap_rosbag <pcap> <bag> \\
    --ros-args -p dump_path:=/tmp/dump -p auto_quit:=true
  ROS_DOMAIN_ID=99 ros2 run glim_ros offline_viewer /tmp/dump \\
    --ros-args -p use_sim_time:=true

File: av24.urdf (robot description, URDF)
Before this commit: robot AV 21, 40 links, 39 joints
Links:
- removed link gps_antenna_rear
- removed link gps_bottom
- removed link gps_top
- removed link imu_bottom
- removed link imu_top
- removed link imu_vectornav
- added link gps_antenna_top
- added link novatel_a
- added link novatel_b
- added link pointonenav
Joints:
- removed joint gps_antenna_rear_joint
- removed joint gps_bottom_joint
- removed joint gps_top_joint
- removed joint imu_bottom_joint
- removed joint imu_top_joint
- removed joint imu_vectornav_joint
- added joint gps_antenna_top_joint: type fixed, parent rear_axle_middle, child gps_antenna_top, origin xyz=1.27135 0.0 0.91994
- added joint novatel_a_joint: type fixed, parent rear_axle_middle, child novatel_a, origin xyz=1.636 -0.075 0.101
- added joint novatel_b_joint: type fixed, parent rear_axle_middle, child novatel_b, origin xyz=1.636 0.075 0.101
- added joint pointonenav_joint: type fixed, parent rear_axle_middle, child pointonenav, origin xyz=1.898 0.027 0.450
- joint camera_front_joint: origin xyz=1.473 -0.140 0.543 rpy=0 0 0 -> xyz=1.365 0.0 0.723 rpy=0 0 0; parent base_link -> rear_axle_middle
- joint camera_front_left_center_joint: origin xyz=2.22226 0.19 0.41974 rpy=0.0 0.0 0.0 -> xyz=2.232 0.180 0.442 rpy=0.0 0.0 0.0; parent base_link -> rear_axle_middle
- joint camera_front_right_center_joint: origin xyz=2.22226 -0.19 0.41974 rpy=0.0 0.0 0.0 -> xyz=2.232 -0.180 0.442 rpy=0.0 0.0 0.0; parent base_link -> rear_axle_middle
- joint camera_left_joint: origin xyz=2.02088 0.17246 0.408 rpy=0 0 1.74533 -> xyz=2.020 0.172 0.418 rpy=0 0 1.74533; parent base_link -> rear_axle_middle
- joint camera_rear_joint: origin xyz=1.473 0.140 0.543 rpy=0 0 3.14159 -> xyz=1.215 0.0 0.723 rpy=0 0 3.14159265358979; parent base_link -> rear_axle_middle
- joint camera_right_joint: origin xyz=2.02088 -0.17190 0.408 rpy=0 0 -1.74533 -> xyz=2.020 -0.172 0.418 rpy=0 0 -1.74533; parent base_link -> rear_axle_middle
- joint fl_tyre_joint: origin xyz=0.0 0.91045 0.0 rpy=0 0 1.5708 -> xyz=0.0 0.91045 0.0 rpy=0 0 0.0
- joint fr_tyre_joint: origin xyz=0.0 -0.91045 0.0 rpy=0 0 1.5708 -> xyz=0.0 -0.91045 0.0 rpy=0 0 0.0
- joint gps_antenna_front_joint: origin xyz=3.17566 0.00005 0.37202 -> xyz=3.17566 0.00005 0.352; parent base_link -> rear_axle_middle
- joint gps_antenna_left_joint: parent base_link -> rear_axle_middle
- joint gps_antenna_right_joint: parent base_link -> rear_axle_middle
- joint luminar_front_joint: origin xyz=2.22177 0.00541 0.46683 rpy=0.0 0.0 0.0 -> xyz=2.222 0.005 0.448 rpy=0.0 0.0 0.0; parent base_link -> rear_axle_middle
- joint luminar_left_joint: origin xyz=1.56355 0.14878 0.53550 rpy=0.0 0.0 1.9634954 -> xyz=1.564 0.149 0.535 rpy=0.0 0.0 1.9634954 ; parent base_link -> rear_axle_middle
- joint luminar_rear_joint: origin xyz=-0.42919 -0.00541 0.21343 rpy=0.0 0.0 3.14159 -> xyz=-0.429 -0.0045 0.217 rpy=0.0 0.0 3.14159265358979; parent base_link -> rear_axle_middle
- joint luminar_right_joint: origin xyz=1.66919 -0.15292 0.53550 rpy=0.0 0.0 -1.9634954 -> xyz=1.574 -0.153 0.535 rpy=0.0 0.0 -1.9634954 ; parent base_link -> rear_axle_middle
- joint model_joint: origin xyz=1.725 0.0 -0.31 rpy=1.5708 0.0 1.5708 -> xyz=1.725 0.0 -0.31 rpy=0.0 0.0 1.5708
- joint radar_front_joint: origin xyz=1.78938 0.0 0.57802 -> xyz=1.789 0.0 0.578; parent base_link -> rear_axle_middle
- joint radar_rear_joint: origin xyz=-0.75249 0.0 0.10652 rpy=0 0 3.14159265358979 -> xyz=-0.752 0.0 0.107 rpy=0 0 3.14159265358979; parent base_link -> rear_axle_middle
- joint rl_tyre_joint: origin xyz=0.00238 0.83734 0.03456 rpy=0 0 1.5708 -> xyz=0.00238 0.83734 0.03456 rpy=0 0 0.0
- joint rr_tyre_joint: origin xyz=0.00194 -0.83734 0.0344 rpy=0 0 1.5708 -> xyz=0.00194 -0.83734 0.0344 rpy=0 0 0.0
- joint vectornav_joint: origin xyz=1.77099 0.0 -0.11125 -> xyz=1.754 0.0 0.118; parent base_link -> rear_axle_middle
